File: board/ssr-channel.kicad_sch (KiCad schematic)
At the start: 9 parts, among them J1 ${Channel}, U4 MOC306XMS

Commit message: WIP
Parts:
- removed D2: LED, LED_SMD:LED_0805_2012Metric_Pad1.15x1.40mm_HandSolder, symbol Device:LED
- removed J1: ${Channel}, Connector_Phoenix_MSTB:PhoenixContact_MSTBA_2,5_3-G_1x03_P5.00mm_Horizontal, symbol Connector_Generic:Conn_01x03
- removed R3: 330R, Resistor_SMD:R_0805_2012Metric, symbol Device:R
- renumbered R4 to R3, R5 to R4, R6 to R5, R7 to R6
Connections:
- net MAINS-L: now also D3.2 (A2), R5.2, R6.1; no longer D3.1 (A1), R4.2
- net ~{CH${Channel}} renamed ~{IN}
- new net OUT: D3.1 (A1), R4.2
Other:
- moved on the sheet: R3
