File: board/CPG.kicad_pcb (KiCad board)
At the start: 2 copper layers, 60 x 62 mm, 39 parts, among them J1 MAINS, J2 VALVE, J3 PUMP, U1 PAN2110P0AA, U2 PY32F030F1xPx, U3 HLK-PM03, U4 MOC306XMS, U5 MOC306XMS, U6 MOC306XMS, X1 SWD, Y1 16MHz

Commit message: Add CPG firmware and correct SWD header
Connections:
- U2 pad 13: Net-(U2-PA11) -> unconnected-(U2-PA11-Pad13)
- U2 pad 15: unconnected-(U2-PA14-Pad15) -> Net-(U2-PA14)
- X1 pad 1: Net-(U2-PA11) -> Net-(U2-PA13)
- X1 pad 3: Net-(U2-PA13) -> Net-(U2-PA14)
Routing:
- net Net-(U2-PA14): track 0.00 -> 24.0 mm, vias 0 -> 2
- net Net-(U2-PA11): track 19.1 -> 0.00 mm, vias 2 -> 0
- net Net-(U2-PA13): track 23.3 -> 19.8 mm
Other:
- board text added: "bleriot-CPG v1.1 drake.cz"
- board text removed: "bleriot-CPG v1.0 drake.cz"
Changed lines of the file:
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@@
 			(unit
 				(name "A")
-				(pins "1" "2" "3")
+				(pins "1" "3" "2")
 			)
 		)
@@
 			(layers "*.Cu" "*.Mask" "F.SilkS")
 			(remove_unused_layers no)
-			(net "Net-(U2-PA11)")
-			(pinfunction "SWDIO_1")
+			(net "Net-(U2-PA13)")
+			(pinfunction "DIO_1")
 			(pintype "bidirectional")
 		)
@@
 			(layers "*.Cu" "*.Mask" "F.SilkS")
 			(remove_unused_layers no)
-			(net "Net-(U2-PA13)")
-			(pinfunction "SWCLK_3")
+			(net "Net-(U2-PA14)")
+			(pinfunction "CLK_3")
 			(pintype "bidirectional")
 		)
@@
 			(layers "F.Cu" "F.Mask" "F.Paste")
 			(roundrect_rratio 0.25)
-			(net "Net-(U2-PA11)")
+			(net "unconnected-(U2-PA11-Pad13)")
 			(pinfunction "PA11_13")
-			(pintype "bidirectional")
+			(pintype "bidirectional+no_connect")
 		)
 		(pad "14" smd roundrect
@@
 			(layers "F.Cu" "F.Mask" "F.Paste")
 			(roundrect_rratio 0.25)
-			(net "unconnected-(U2-PA14-Pad15)")
+			(net "Net-(U2-PA14)")
 			(pinfunction "PA14_15")
-			(pintype "bidirectional+no_connect")
+			(pintype "bidirectional")
 		)
 		(pad "16" smd roundrect
@@
 			(net "unconnected-(U2-PF4-BOOT0-Pad20)")
 			(pinfunction "PF4-BOOT0_20")
-			(pintype "bidirectional")
+			(pintype "bidirectional+no_connect")
 		)
 		(embedded_fonts no)
@@
 		(layer "Edge.Cuts")
 	)
-	(gr_text "bleriot-CPG v1.0 drake.cz"
+	(gr_text "bleriot-CPG v1.1 drake.cz"
 		(at 83 79 90)
 		(layer "F.SilkS")
@@
 		(width 0.4)
 		(layer "F.Cu")
-		(net "Net-(U2-PA11)")
-	)
-	(segment
-		(start 102.625 95.875)
-		(end 102.625 97.1375)
-		(width 0.4)
-		(layer "F.Cu")
-		(net "Net-(U2-PA11)")
-	)
-	(segment
-		(start 104 95.300003)
-		(end 103.899997 95.2)
-		(width 0.4)
-		(layer "F.Cu")
-		(net "Net-(U2-PA11)")
-	)
-	(segment
-		(start 103.3 95.2)
-		(end 102.625 95.875)
-		(width 0.4)
-		(layer "F.Cu")
-		(net "Net-(U2-PA11)")
-	)
-	(segment
-		(start 108.800003 95.300003)
-		(end 110.46 96.96)
-		(width 0.4)
-		(layer "F.Cu")
-		(net "Net-(U2-PA11)")
-	)
-	(segment
-		(start 107 95.300003)
-		(end 108.800003 95.300003)
-		(width 0.4)
-		(layer "F.Cu")
-		(net "Net-(U2-PA11)")
-	)
-	(segment
-		(start 103.899997 95.2)
-		(end 103.3 95.2)
-		(width 0.4)
-		(layer "F.Cu")
-		(net "Net-(U2-PA11)")
-	)
-	(via
-		(at 107 95.300003)
-		(size 0.6)
-		(drill 0.4)
-		(layers "F.Cu" "B.Cu")
-		(net "Net-(U2-PA11)")
-	)
-	(via
-		(at 104 95.300003)
-		(size 0.6)
-		(drill 0.4)
-		(layers "F.Cu" "B.Cu")
-		(net "Net-(U2-PA11)")
-	)
-	(segment
-		(start 107 95.300003)
-		(end 104 95.300003)
-		(width 0.4)
-		(layer "B.Cu")
-		(net "Net-(U2-PA11)")
-	)
-	(segment
-		(start 104 94.5)
-		(end 103 94.5)
-		(width 0.4)
-		(layer "F.Cu")
 		(net "Net-(U2-PA13)")
 	)
 	(segment
-		(start 101.975 95.525)
-		(end 101.975 97.1375)
+		(start 102.449997 95.300003)
+		(end 104 95.300003)
 		(width 0.4)
 		(layer "F.Cu")
@@
 	)
 	(segment
-		(start 103 94.5)
-		(end 101.975 95.525)
+		(start 101.975 97.1375)
+		(end 101.975 95.775)
 		(width 0.4)
 		(layer "F.Cu")
@@
 	)
 	(segment
-		(start 115.54 101.04)
-		(end 115.54 106)
+		(start 108.800003 95.300003)
+		(end 110.46 96.96)
 		(width 0.4)
 		(layer "F.Cu")
@@
 	)
 	(segment
-		(start 109 94.5)
-		(end 115.54 101.04)
+		(start 107 95.300003)
+		(end 108.800003 95.300003)
 		(width 0.4)
 		(layer "F.Cu")
@@
 	)
 	(segment
-		(start 107 94.5)
-		(end 109 94.5)
+		(start 101.975 95.775)
+		(end 102.449997 95.300003)
 		(width 0.4)
 		(layer "F.Cu")
@@
 	)
 	(via
-		(at 104 94.5)
+		(at 107 95.300003)
 		(size 0.6)
 		(drill 0.4)
@@
 	)
 	(via
-		(at 107 94.5)
+		(at 104 95.300003)
 		(size 0.6)
 		(drill 0.4)
@@
 	)
 	(segment
-		(start 107 94.5)
-		(end 104 94.5)
+		(start 107 95.300003)
+		(end 104 95.300003)
 		(width 0.4)
 		(layer "B.Cu")
@@
 		(net "/VALVE_CW")
 	)
+	(segment
+		(start 101.325 95.425)
+		(end 101.325 97.1375)
+		(width 0.4)
+		(layer "F.Cu")
+		(net "Net-(U2-PA14)")
+	)
+	(segment
+		(start 115.54 101.04)
+		(end 115.54 106)
+		(width 0.4)
+		(layer "F.Cu")
+		(net "Net-(U2-PA14)")
+	)
+	(segment
+		(start 102.25 94.5)
+		(end 101.325 95.425)
+		(width 0.4)
+		(layer "F.Cu")
+		(net "Net-(U2-PA14)")
+	)
+	(segment
+		(start 109 94.5)
+		(end 115.54 101.04)
+		(width 0.4)
+		(layer "F.Cu")
+		(net "Net-(U2-PA14)")
+	)
+	(segment
+		(start 107 94.5)
+		(end 109 94.5)
+		(width 0.4)
+		(layer "F.Cu")
+		(net "Net-(U2-PA14)")
+	)
+	(segment
+		(start 104 94.5)
+		(end 102.25 94.5)
+		(width 0.4)
+		(layer "F.Cu")
+		(net "Net-(U2-PA14)")
+	)
+	(via
+		(at 104 94.5)
+		(size 0.6)
+		(drill 0.4)
+		(layers "F.Cu" "B.Cu")
+		(net "Net-(U2-PA14)")
+	)
+	(via
+		(at 107 94.5)
+		(size 0.6)
+		(drill 0.4)
+		(layers "F.Cu" "B.Cu")
+		(net "Net-(U2-PA14)")
+	)
+	(segment
+		(start 107 94.5)
+		(end 104 94.5)
+		(width 0.4)
+		(layer "B.Cu")
+		(net "Net-(U2-PA14)")
+	)
 	(zone
