File: board/CPG.kicad_sch (KiCad schematic)
At the start: 20 parts, among them U1 PAN2110P0AA, U2 HLK-PM03, U3 PY32F030K1xTx, X1 SWD, Y1 16MHz

Commit message: WIP
Parts:
- removed C5, C7: 100n, Capacitor_SMD:C_0805_2012Metric, symbol Device:C
- removed IN1: MAINS, Connector_Phoenix_MSTB:PhoenixContact_MSTBA_2,5_3-G_1x03_P5.00mm_Horizontal, symbol Connector_Generic:Conn_01x03
- removed U3: PY32F030K1xTx, Package_QFP:LQFP-32_7x7mm_P0.8mm, symbol MCU_Puya_PY32F:PY32F030K1xTx
- added C4: 100n, Capacitor_SMD:C_0805_2012Metric, symbol Device:C
- added D1: WS2812B, LED_SMD:LED_WS2812B_PLCC4_5.0x5.0mm_P3.2mm, symbol LED:WS2812B
- added J1: MAINS, Connector_Phoenix_MSTB:PhoenixContact_MSTBA_2,5_3-G_1x03_P5.00mm_Horizontal, symbol Connector:Conn_01x03_Pin
- added J2: VALVE, Connector_Phoenix_MSTB:PhoenixContact_MSTBA_2,5_3-G_1x03_P5.00mm_Horizontal, symbol Connector:Conn_01x03_Pin
- added J3: PUMP, Connector_Phoenix_MSTB:PhoenixContact_MSTBA_2,5_3-G_1x03_P5.00mm_Horizontal, symbol Connector:Conn_01x03_Pin
- added U2: PY32F030F1xPx, Package_SO:TSSOP-20_4.4x6.5mm_P0.65mm, symbol MCU_Puya_PY32F:PY32F030F1xPx
- D2: renamed from D1; now not fitted
- R2: now not fitted
- renumbered C4 to C5, U2 to U3
Connections:
- net +3V3: now also D1.1 (VDD), U2.9 (VCC)
- net GND: now also R2.1, C4.2, D1.3 (VSS), U2.7 (VSS); no longer D2.1 (K)
- net LED: now also D2.2 (A), D1.4 (DIN), U2.19 (PB7); no longer R2.2
- net MAINS-L: now also J1.3 (Pin_3)
- net MAINS-N: now also J1.2 (Pin_2), J2.1 (Pin_1), J3.1 (Pin_1)
- net MAINS-PE: now also J1.1 (Pin_1), J3.3 (Pin_3)
- net RF_DATA: now also U2.6 (PA3)
- net RF_SCK: now also U2.5 (PA2)
- net ~{RF_CS}: now also U2.4 (PF3)
- net at X1.1 (SWDIO): now also U2.13 (PA11)
- net at X1.3 (SWCLK): now also U2.14 (PA13)
- new net: D2.1 (K), R2.2
- new net: C4.1, U2.3 (PF2-NRST)
- new net PUMP: U2.16 (PB4)
- new net VALVE_CCW: U2.17 (PB5)
- new net VALVE_CW: U2.18 (PB6)
- new net pump/OUT: J3.2 (Pin_2)
- new net valve-ccw/OUT: J2.2 (Pin_2)
- new net valve-cw/OUT: J2.3 (Pin_3)
- no-connect marks 16 -> 8
Other:
- sheet channel1 renamed valve-cw
- removed sheet channel2
- removed sheet channel3
- removed sheet channel4
- removed sheet channel5
- added sheet pump (ssr-channel.kicad_sch)
- added sheet valve-ccw (ssr-channel.kicad_sch)
- sheet valve-cw ports: added OUT, ~{IN}; removed none
- moved on the sheet: C3, C5

Commit message: WIP
Parts:
- removed H2: MountingHole, MountingHole:MountingHole_3.7mm_Pad_Via, symbol Mechanical:MountingHole
Connections:
- net MAINS-N: now also J3.2 (Pin_2); no longer J3.1 (Pin_1)
- net MAINS-PE: now also J3.1 (Pin_1); no longer J3.3 (Pin_3)
- net pump/OUT: now also J3.3 (Pin_3); no longer J3.2 (Pin_2)
Other:
- moved on the sheet: J3
Changed lines of the file:
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@@
 	(global_label "MAINS-PE"
 		(shape input)
-		(at 110.49 158.75 180)
+		(at 110.49 166.37 180)
 		(fields_autoplaced yes)
 		(effects
@@
 		)
 		(property "Intersheetrefs" "${INTERSHEET_REFS}"
-			(at 96.0817 158.75 0)
+			(at 96.0817 166.37 0)
 			(hide yes)
 			(show_name no)
@@
 	)
 	(symbol
-		(lib_id "Mechanical:MountingHole")
-		(at 245.11 152.4 0)
-		(unit 1)
-		(body_style 1)
-		(exclude_from_sim no)
-		(in_bom yes)
-		(on_board yes)
-		(in_pos_files yes)
-		(dnp no)
-		(fields_autoplaced yes)
-		(property "Reference" "H2"
-			(at 247.65 151.8055 0)
-			(show_name no)
-			(do_not_autoplace no)
-			(effects
-				(font
-					(size 1.27 1.27)
-				)
-				(justify left)
-			)
-		)
-		(property "Value" "MountingHole"
-			(at 247.65 153.5677 0)
-			(show_name no)
-			(do_not_autoplace no)
-			(effects
-				(font
-					(size 1.27 1.27)
-				)
-				(justify left)
-			)
-		)
-		(property "Footprint" "MountingHole:MountingHole_3.7mm_Pad_Via"
-			(at 245.11 152.4 0)
-			(hide yes)
-			(show_name no)
-			(do_not_autoplace no)
-			(effects
-				(font
-					(size 1.27 1.27)
-				)
-			)
-		)
-		(property "Datasheet" ""
-			(at 245.11 152.4 0)
-			(hide yes)
-			(show_name no)
-			(do_not_autoplace no)
-			(effects
-				(font
-					(size 1.27 1.27)
-				)
-			)
-		)
-		(property "Description" "Mounting Hole without connection"
-			(at 245.11 152.4 0)
-			(hide yes)
-			(show_name no)
-			(do_not_autoplace no)
-			(effects
-				(font
-					(size 1.27 1.27)
-				)
-			)
-		)
-		(instances
-			(project "CPG"
-				(path "/6b7dd4b9-634f-41b4-b846-9b2e2d6d43c6"
-					(reference "H2")
-					(unit 1)
-				)
-			)
-		)
-	)
-	(symbol
 		(lib_id "Device:C")
 		(at 163.83 107.95 0)
@@
 	(symbol
 		(lib_id "Connector:Conn_01x03_Pin")
-		(at 115.57 161.29 180)
+		(at 115.57 163.83 180)
 		(unit 1)
 		(body_style 1)
@@
 		(fields_autoplaced yes)
 		(property "Reference" "J3"
-			(at 116.84 160.0199 0)
+			(at 116.84 162.5599 0)
 			(show_name no)
 			(do_not_autoplace no)
@@
 		)
 		(property "Value" "PUMP"
-			(at 116.84 162.5599 0)
+			(at 116.84 165.0999 0)
 			(show_name no)
 			(do_not_autoplace no)
@@
 		)
 		(property "Footprint" "Connector_Phoenix_MSTB:PhoenixContact_MSTBA_2,5_3-G_1x03_P5.00mm_Horizontal"
-			(at 115.57 161.29 0)
-			(hide yes)
-			(show_name no)
-			(do_not_autoplace no)
-			(effects
-				(font
-					(size 1.27 1.27)
-				)
-			)
-		)
-		(property "Datasheet" ""
-			(at 115.57 161.29 0)
+			(at 115.57 163.83 0)
+			(hide yes)
+			(show_name no)
+			(do_not_autoplace no)
+			(effects
+				(font
+					(size 1.27 1.27)
+				)
+			)
+		)
+		(property "Datasheet" ""
+			(at 115.57 163.83 0)
 			(hide yes)
 			(show_name no)
@@
 		)
 		(property "Description" "Generic connector, single row, 01x03, script generated"
-			(at 115.57 161.29 0)
-			(hide yes)
-			(show_name no)
+			(at 115.57 163.83 0)
+			(hide yes)
+			(show_name no)
